File: PCBs/switch_main_v1/mcu.kicad_sch (KiCad schematic)
At the start: 3 parts, among them U301 M24256X-FCU6T_VF, U302 STM32H573RIVx

Commit message: Changed MCU to STM32H573VIT3Q
Parts:
- removed U302: STM32H573RIVx, switch_footprints:QFN-68-1EP_8x8mm_P0.4mm_EP6.4x6.4mm, symbol STM32H573RIV:STM32H573RIVx
- added C301: 220p, Capacitor_SMD:C_0402_1005Metric, symbol Device:C_Small
- added C302, C306, C310, C314, C317, C318, C322, C326: 100n, Capacitor_SMD:C_0402_1005Metric, symbol Device:C_Small
- added C303, C321: 1u, Capacitor_SMD:C_0402_1005Metric, symbol Device:C_Small
- added C304, C309, C313, C330: 4u7, Capacitor_SMD:C_0402_1005Metric, symbol Device:C_Small
- added C305: 10u, Capacitor_SMD:C_0402_1005Metric, symbol Device:C_Small
- added C307, C308, C311, C316: 10n, Capacitor_SMD:C_0402_1005Metric, symbol Device:C_Small
- added C312, C315: 6p, Capacitor_SMD:C_0402_1005Metric, symbol Device:C_Small
- added D301: Red, LED_SMD:LED_0402_1005Metric, symbol Device:LED_Small
- added D302: Green, LED_SMD:LED_0402_1005Metric, symbol Device:LED_Small
- added D303: Blue, LED_SMD:LED_0402_1005Metric, symbol Device:LED_Small
- added L301: 2u2, Inductor_SMD:L_Murata_DFE201610P, symbol Device:L_Small
- added R302, R303, R309: 10k, Resistor_SMD:R_0402_1005Metric, symbol Device:R_Small
- added R304: 100k, Resistor_SMD:R_0402_1005Metric, symbol Device:R_Small
- added R305: 4k7, Resistor_SMD:R_0402_1005Metric, symbol Device:R_Small
- added R306, R307, R308: 2k7, Resistor_SMD:R_0402_1005Metric, symbol Device:R_Small
- added S301, S302, S303, S304: TS20-42-25-WT-160-SMT-TR, switch_footprints:TS204225WT160SMTTRMSL, symbol TS20-42-25-WT-160-SMT-TR-MSL:TS20-42-25-WT-160-SMT-TR
- added U302: STM32H573VIT3Q, switch_footprints:QFP50P1600X1600X160-100N, symbol STM32H573VIT3Q:STM32H573VIT3Q
- added Y301: ECS-250-10-36Q-AES-TR, Crystal:Crystal_SMD_2520-4Pin_2.5x2.0mm, symbol Device:Crystal_GND24_Small
Connections:
- net +2V5: now also U301.A1 (VCC), C302.1, C303.1, C304.1, C305.1, C306.2, C310.2, C314.2, C318.2, C322.2, C326.2, C330.2, R302.2, R303.2, R309.2, U302.100 (VDD), U302.11 (VDD), U302.21 (VDDA), U302.27 (VDD), U302.47 (VDDSMPS), U302.51 (VDD), U302.6 (VBAT), U302.73 (VDDUSB), U302.75 (VDD)
- net ETHERNET_RST: now also C308.1, R302.1, S302.2 (NO_2)
- net ETH_PPS_OUT: now also U302.91 (PB5)
- net GND: now also U301.B2 (VSS), C301.2, C302.2, C303.2, C304.2, C305.2, C306.1, C307.2, C308.2, C309.2, C310.1, C311.2, C312.2, C313.2, C314.1, C315.2, C316.2, C317.2, C318.1, C321.2, C322.1, C326.1, C330.1, R305.2, R306.1, R307.1, R308.1, S301.3 (COM_1), S302.3 (COM_1), S303.3 (COM_1), S304.3 (COM_1), U302.10 (VSS), U302.19 (VSSA), U302.26 (VSS), U302.48 (VSSSMPS), U302.50 (VSS), U302.74 (VSS), U302.99 (VSS), Y301.2, Y301.4
- net MCO1: now also U302.67 (PA8)
- net RST: now also C307.1, S301.2 (NO_2), U302.14 (NRST)
- net I3C1_SCL: now reaches U301.A2 (SCL)
- net I3C1_SDA: now reaches U301.B1 (SDA)
- new net +VIN: R304.1
- new net BOOT: C316.1, R309.1, S304.2 (NO_2), U302.94 (BOOT0)
- new net BTN: C311.1, R303.1, S303.2 (NO_2)
- new net LEDB: D303.2 (A)
- new net LEDB_K: D303.1 (K), R308.2
- new net LEDG: D302.2 (A)
- new net LEDG_K: D302.1 (K), R307.2
- new net LEDR: D301.2 (A)
- new net LEDR_K: D301.1 (K), R306.2
- new net OSC_IN: C312.1, U302.12 (PH0), Y301.3
- new net OSC_OUT: C315.1, U302.13 (PH1), Y301.1
- new net VCAP: C309.1, C313.1, L301.2, U302.49 (VCAP), U302.98 (VCAP)
- new net VIN_ADC: R304.2, R305.1
- new net VLXSMPS: C301.1, L301.1, U302.46 (VLXSMPS)
- new net VREF+: C317.1, C321.1, U302.20 (VREF+)
- no-connect marks 0 -> 8
Other:
- note added: "Buttons, LEDs, oscillator, pullups, EEPROM, ADC battery input"
- note added: "VCAP"
- note added: "VDD"
- note added: "VDDA"
- note added: "VDDSMPS"
- note added: "VREF+"
- note removed: "Buttons, LEDs, oscillator, pullups, EEPROM"
- moved on the sheet: R301, U301

Commit message: Changed MCU to STM32H573IIK3Q
Parts:
- removed S304: TS20-42-25-WT-160-SMT-TR, switch_footprints:TS204225WT160SMTTRMSL, symbol TS20-42-25-WT-160-SMT-TR-MSL:TS20-42-25-WT-160-SMT-TR
- removed U302: STM32H573VIT3Q, switch_footprints:QFP50P1600X1600X160-100N, symbol STM32H573VIT3Q:STM32H573VIT3Q
- added C319, C320, C323, C324, C325: 100n, Capacitor_SMD:C_0402_1005Metric, symbol Device:C_Small
- added S305: PCM12SMTR, switch_footprints:PCM12SMTR, symbol PCM12SMTR:PCM12SMTR
- added U302: STM32H573IIK3Q, switch_footprints:STM32H573IIK3Q, symbol STM32H573IIK3Q:STM32H573IIK3Q
- C316: value 10n -> 100n
- R309: value 10k -> 1k
Connections:
- net +2V5: now also C316.2, C319.2, C320.2, C323.2, C324.2, C325.2, S305.1 (A), U302.B1 (VBAT), U302.D10 (VDD), U302.D5 (VDD), U302.D7 (VDDIO2), U302.D8 (VDD), U302.E12 (VDD), U302.E4 (VDD), U302.F12 (VDDUSB), U302.H4 (VDD), U302.J12 (VDD), U302.L4 (VDD), U302.M1 (VDDA), U302.M11 (VDD), U302.M6 (VDD), U302.M8 (VDD), U302.R13 (VDDSMPS); no longer R309.2
- net BOOT: now also U302.A5 (BOOT0); no longer C316.1
- net CAN.RXD: now also U302.D15 (PA11)
- net CAN.TXD: now also U302.C15 (PA12)
- net ETH_PPS_OUT: now also U302.A6 (PB5)
- net GND: now also C316.1, C319.1, C320.1, C323.1, C324.1, C325.1, S305.3 (C), U302.C1 (VSS), U302.D11 (VSS), U302.D14 (VSS), U302.D6 (VSS), U302.D9 (VSS), U302.F10 (VSS), U302.F6 (VSS), U302.F7 (VSS), U302.F8 (VSS), U302.F9 (VSS), U302.G10 (VSS), U302.G12 (VSS), U302.G4 (VSS), U302.G6 (VSS), U302.G7 (VSS), U302.G8 (VSS), U302.G9 (VSS), U302.H10 (VSS), U302.H12 (VSS), U302.H6 (VSS), U302.H7 (VSS), U302.H8 (VSS), U302.H9 (VSS), U302.J10 (VSS), U302.J6 (VSS), U302.J7 (VSS), U302.J8 (VSS), U302.J9 (VSS), U302.K1 (VSS), U302.K10 (VSS), U302.K6 (VSS), U302.K7 (VSS), U302.K8 (VSS), U302.K9 (VSS), U302.M2 (VSSA), U302.M4 (VSS), U302.M7 (VSS), U302.M9 (VSS), U302.N2 (VREF-), U302.P12 (VSSSMPS); no longer C316.2
- net MCO1: now also U302.F15 (PA8)
- net OSC_IN: now also U302.J1 (PH0)
- net OSC_OUT: now also U302.J2 (PH1)
- net RMII.CRS_DV: now also U302.R4 (PA7)
- net RMII.REF_CLK: now also U302.L3 (PA1)
- net RMII.RX_D0: now also U302.N4 (PC4)
- net RMII.RX_D1: now also U302.P4 (PC5)
- net RMII.TX_D0: now also U302.C8 (PG13)
- net RMII.TX_D1: now also U302.A8 (PG14)
- net RMII.TX_EN: now also U302.C9 (PG11)
- net RST: now also U302.K3 (NRST)
- net SMI.MDC: now also U302.L2 (PC1)
- net SMI.MDIO: now also U302.M3 (PA2)
- net SWD.SWCLK: now also U302.B13 (PA14(JTCK)
- net SWD.SWDIO: now also U302.E13 (PA13(JTMS)
- net SWD.SWO: now also U302.B7 (PB3(JTDO)
- net VCAP: now also U302.A3 (VCAP), U302.R14 (VCAP)
- net VLXSMPS: now also U302.R12 (VLXSMPS)
- net VREF+: now also U302.N1 (VREF+)
- net I3C1_SCL renamed I2C4_SCL
- net I2C4_SCL: now also U302.P15 (PH11)
- net I3C1_SDA renamed I2C4_SDA
- net I2C4_SDA: now also U302.L15 (PD13)
- new net Earth: S305.MP1, S305.MP2, S305.MP3, S305.MP4
- new net SW_COM: R309.2, S305.2 (B)
- no-connect marks 8 -> 6
Other:
- moved on the sheet: C301, C302, C303, C304, C305, C306, C307, C308, C309, C310, C311, C312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
